Commit message: update

File: src/robot_arm_description/urdf/robot/arm.urdf (robot description, URDF)
Before this commit: robot robot_arm, 8 links, 7 joints
Joints:
- joint joint_5: axis 0.650673886413552 0.759313420493717 0.00816229119891543 -> -0.759313420493717 0.650673886413552 0.00816229119891543

Commit message: fixed joint 5

File: src/robot_arm_description/urdf/robot/arm.urdf (robot description, URDF)
Before this commit: robot robot_arm, 8 links, 7 joints
Joints:
- joint joint_5: axis -0.759313420493717 0.650673886413552 0.00816229119891543 -> -0.7748550616 0.6320449991 0.00816229119891543; origin xyz=0.0658770416469138 0.0497166404170352 0.006958042593945 rpy=0 0 0 -> xyz=0.001935 -0.026272 -0.004657 rpy=0 0 0

Commit message: fixed joint 6

File: src/robot_arm_description/urdf/robot/arm.urdf (robot description, URDF)
Before this commit: robot robot_arm, 8 links, 7 joints
Joints:
- joint joint_6: origin xyz=0 0 0 rpy=0 0 0 -> xyz=0.0639420416 0.0759886404 0.0116150426 rpy=0 0 0
