Commit message: hardware test 1

File: src/robot_arm_description/urdf/control/robot_arm_ros2_control.urdf.xacro (robot description, xacro)
@@ -1,4 +1,8 @@
 <?xml version="1.0" ?>
 <robot xmlns:xacro="http://wiki.ros.org/xacro">
+    <!-- ESP32 Connection Parameters (set these to match your setup) -->
+    <xacro:property name="esp32_ip" value="192.168.1.100"/>
+    <xacro:property name="esp32_port" value="5000"/>
+    <xacro:property name="use_simulation" value="true"/>
     <xacro:macro name="robot_arm_ros2_control" params="prefix flange_link use_gazebo">
         <ros2_control name="RobotSystem" type="system">
@@ -9,7 +13,9 @@
                 <xacro:unless value="${use_gazebo}">
                     <plugin>custom_hardware/CustomHardwareInterface</plugin>
-                    <param name="serial_port">/dev/ttyUSB0</param>
-                    <param name="baud_rate">115200</param>
-                    <param name="timeout_ms">1000</param>
+                    <!-- ESP32 WiFi/TCP connection parameters -->
+                    <param name="esp32_ip">${esp32_ip}</param>
+                    <param name="esp32_port">${esp32_port}</param>
+                    <param name="timeout_ms">100</param>
+                    <param name="use_simulation">${use_simulation}</param>
                 </xacro:unless>
             </hardware>

Commit message: hardware test2

File: src/robot_arm_description/urdf/control/robot_arm_ros2_control.urdf.xacro (robot description, xacro)
@@ -2,7 +2,7 @@
 <robot xmlns:xacro="http://wiki.ros.org/xacro">
     <!-- ESP32 Connection Parameters (set these to match your setup) -->
-    <xacro:property name="esp32_ip" value="192.168.1.100"/>
+    <xacro:property name="esp32_ip" value="172.20.10.4"/>
     <xacro:property name="esp32_port" value="5000"/>
-    <xacro:property name="use_simulation" value="true"/>
+    <xacro:property name="use_simulation" value="false"/>
     <xacro:macro name="robot_arm_ros2_control" params="prefix flange_link use_gazebo">
         <ros2_control name="RobotSystem" type="system">

File: src/robot_arm_description/urdf/robot/arm.urdf.xacro (robot description, xacro)
@@ -12,13 +12,14 @@
     <!-- Import arm urdf file -->
     <xacro:include filename="$(find robot_arm_description)/urdf/robot/arm.urdf" />
-    <!-- Include ROS 2 control configuration for Gazebo -->
+    <!-- Include ROS 2 control configuration -->
+    <xacro:include filename="$(find robot_arm_description)/urdf/control/robot_arm_ros2_control.urdf.xacro" />
+    <!-- Load ROS 2 control macro (works for both Gazebo and real hardware) -->
+    <xacro:robot_arm_ros2_control
+        prefix="$(arg prefix)"
+        flange_link="$(arg flange_link)"
+        use_gazebo="$(arg use_gazebo)"/>
+    <!-- Include Gazebo-specific plugins only when using Gazebo -->
     <xacro:if value="$(arg use_gazebo)">
-        <xacro:include filename="$(find robot_arm_description)/urdf/control/robot_arm_ros2_control.urdf.xacro" />
         <xacro:include filename="$(find robot_arm_description)/urdf/control/gazebo_sim_ros2_control.urdf.xacro" />
-        <!-- Load ROS 2 control macro -->
-        <xacro:robot_arm_ros2_control
-            prefix="$(arg prefix)"
-            flange_link="$(arg flange_link)"
-            use_gazebo="$(arg use_gazebo)"/>
         <!-- Load Gazebo ROS 2 control plugin -->
         <xacro:load_gazebo_sim_ros2_control_plugin

Commit message: moveit to hardware

File: src/robot_arm_description/urdf/control/robot_arm_ros2_control.urdf.xacro (robot description, xacro)
@@ -4,6 +4,5 @@
     <xacro:property name="esp32_ip" value="172.20.10.4"/>
     <xacro:property name="esp32_port" value="5000"/>
-    <xacro:property name="use_simulation" value="false"/>
-    <xacro:macro name="robot_arm_ros2_control" params="prefix flange_link use_gazebo">
+    <xacro:macro name="robot_arm_ros2_control" params="prefix flange_link use_gazebo use_simulation:=false">
         <ros2_control name="RobotSystem" type="system">
             <hardware>

File: src/robot_arm_description/urdf/robot/arm.urdf.xacro (robot description, xacro)
@@ -10,4 +10,5 @@
     <xacro:arg name="use_camera" default="false"/>
     <xacro:arg name="use_gazebo" default="false"/>
+    <xacro:arg name="use_simulation" default="false"/>
     <!-- Import arm urdf file -->
     <xacro:include filename="$(find robot_arm_description)/urdf/robot/arm.urdf" />
@@ -18,5 +19,6 @@
         prefix="$(arg prefix)"
         flange_link="$(arg flange_link)"
-        use_gazebo="$(arg use_gazebo)"/>
+        use_gazebo="$(arg use_gazebo)"
+        use_simulation="$(arg use_simulation)"/>
     <!-- Include Gazebo-specific plugins only when using Gazebo -->
     <xacro:if value="$(arg use_gazebo)">
